File: carte-meteo-lora-2.kicad_pcb (KiCad board)
At the start: 4 copper layers, 50 x 50 mm, 81 parts, among them J1 USB_C_Receptacle_USB2.0_14P, J2 Conn_Coaxial, J3 Conn_Coaxial, J4 Conn_Coaxial, J5 Conn_01x04_Pin, SW1 SW_Push, SW2 SW_Push, U1 HS96L03W2C03, U2 SX1262TR8-GC, U3 LDL212PV33R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

Commit message: pcb: add inital layout
Parts:
- removed C13: 0p3, Capacitor_SMD:C_0402_1005Metric
- removed H2: MountingHole_Pad, MountingHole:MountingHole_2.2mm_M2_Pad_Via
- moved H1 57.6 mm to (140.0, 33.0)
- moved U1 49.1 mm to (106.0, 50.6)
- moved D3 45.9 mm to (129.0, 75.2)
- moved C1 44.5 mm to (133.0, 76.5), turned to 90 degrees
- moved TP6 20.3 mm to (105.8, 31.8), turned to 180 degrees
- moved D6 19.7 mm to (135.2, 38.8)
- moved TP3 17.5 mm to (105.8, 34.2), turned to 180 degrees
- moved TP7 17.3 mm to (112.2, 34.9)
- moved TP4 17.1 mm to (109.7, 34.9)
- moved TP11 8.63 mm to (127.1, 33.0)
- moved C11 8.00 mm to (120.5, 30.5)
- moved R9 8.00 mm to (123.0, 30.5)
- moved C2 7.99 mm to (61.4, 64.5)
- moved SW2 7.76 mm to (121.8, 33.0)
- moved C12 6.54 mm to (129.3, 32.8)
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