File: carte-meteo-lora-2.kicad_sch (KiCad schematic)
At the start: 80 parts, among them J1 USB_C_Receptacle_USB2.0_14P, J2 Conn_Coaxial, J3 Conn_Coaxial, J4 Conn_Coaxial, J5 Conn_01x04_Pin, SW1 SW_Push, SW2 SW_Push, U1 HS96L03W2C03, U2 SX1262TR8-GC, U3 LDL212PV33R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

Commit message: pcb: add inital layout
Parts:
- removed H2: MountingHole_Pad, MountingHole:MountingHole_2.2mm_M2_Pad_Via, symbol Mechanical:MountingHole_Pad
Changed lines of the file:
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@@
 	)
 	(junction
-		(at 130.81 161.29)
-		(diameter 0)
-		(color 0 0 0 0)
-	)
-	(junction
 		(at 195.58 54.61)
 		(diameter 0)
@@
 	(wire
 		(pts
-			(xy 130.81 161.29) (xy 130.81 160.02)
-		)
-		(stroke
-			(width 0)
-			(type default)
-		)
-	)
-	(wire
-		(pts
 			(xy 250.19 25.4) (xy 250.19 26.67)
 		)
@@
 	(wire
 		(pts
-			(xy 130.81 161.29) (xy 137.16 161.29)
-		)
-		(stroke
-			(width 0)
-			(type default)
-		)
-	)
-	(wire
-		(pts
 			(xy 82.55 76.2) (xy 82.55 77.47)
 		)
@@
 	(wire
 		(pts
-			(xy 125.73 161.29) (xy 130.81 161.29)
+			(xy 125.73 161.29) (xy 137.16 161.29)
 		)
 		(stroke
@@
 					(unit 1)
 				)
-			)
-		)
-	)
-	(symbol
-		(lib_id "Mechanical:MountingHole_Pad")
-		(at 130.81 157.48 0)
-		(unit 1)
-		(body_style 1)
-		(exclude_from_sim no)
-		(in_bom no)
-		(on_board yes)
-		(in_pos_files yes)
-		(dnp no)
-		(property "Reference" "H2"
-			(at 127.508 158.75 0)
-			(show_name no)
-			(do_not_autoplace no)
-			(effects
-				(font
-					(size 1.27 1.27)
-				)
-				(justify left)
-			)
-		)
-		(property "Value" "MountingHole_Pad"
-			(at 134.62 156.21 90)
-			(hide yes)
-			(show_name no)
-			(do_not_autoplace no)
-			(effects
-				(font
-					(size 1.27 1.27)
-				)
-			)
-		)
-		(property "Footprint" "MountingHole:MountingHole_2.2mm_M2_Pad_Via"
-			(at 130.81 157.48 0)
-			(hide yes)
-			(show_name no)
-			(do_not_autoplace no)
-			(effects
-				(font
-					(size 1.27 1.27)
-				)
-			)
-		)
-		(property "Datasheet" ""
-			(at 130.81 157.48 0)
-			(hide yes)
-			(show_name no)
-			(do_not_autoplace no)
-			(effects
-				(font
-					(size 1.27 1.27)
-				)
-			)
-		)
-		(property "Description" "Mounting Hole with connection"
-			(at 130.81 157.48 0)
-			(hide yes)
-			(show_name no)
-			(do_not_autoplace no)
-			(effects
-				(font
-					(size 1.27 1.27)
-				)
-			)
-		)
-		(pin "1"
-		)
-		(instances
-			(project "carte-meteo-lora-2"
-				(path "/14cd50fe-ec77-4829-bd74-9322c036cdc1"
-					(reference "H2")
-					(unit 1)
-				)

Commit message: pcb: reorganize programmable gpios
Connections:
- net BUSY: now also U4.17 (GPIO8/SDIO_DATA0); no longer U4.19 (GPIO10/SDIO_CMD)
- net DIO1: now also U4.19 (GPIO10/SDIO_CMD); no longer U4.33 (GPIO23)
- net DIO3: now also U4.18 (GPIO9/SDIO_CLK); no longer U4.34 (GPIO24)
- net RGB1: now also U4.34 (GPIO24); no longer U4.17 (GPIO8/SDIO_DATA0)
- net RST: now also U4.33 (GPIO23); no longer U4.18 (GPIO9/SDIO_CLK)

Commit message: pcb: add lora module routing
Connections:
- net BUSY: now also U4.37 (GPIO27); no longer U4.17 (GPIO8/SDIO_DATA0)
- net DIO1: now also U4.35 (GPIO25); no longer U4.19 (GPIO10/SDIO_CMD)
- net DIO3: now also U4.36 (GPIO26); no longer U4.18 (GPIO9/SDIO_CLK)
Other:
- moved on the sheet: R12
Changed lines of the file:
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@@
 	)
 	(no_connect
-		(at 170.18 81.28)
+		(at 236.22 81.28)
 	)
 	(no_connect
-		(at 236.22 119.38)
+		(at 236.22 83.82)
 	)
 	(no_connect
-		(at 114.3 100.33)
+		(at 236.22 78.74)
 	)
 	(no_connect
-		(at 49.53 105.41)
+		(at 170.18 81.28)
 	)
 	(no_connect
-		(at 236.22 114.3)
+		(at 114.3 100.33)
 	)
 	(no_connect
-		(at 87.63 130.81)
+		(at 49.53 105.41)
 	)
 	(no_connect
-		(at 114.3 130.81)
+		(at 87.63 130.81)
 	)
 	(no_connect
-		(at 236.22 116.84)
+		(at 114.3 130.81)
 	)
 	(no_connect
@@
 	(wire
 		(pts
-			(xy 248.92 121.92) (xy 250.19 121.92)
+			(xy 250.19 121.92) (xy 251.46 121.92)
 		)
 		(stroke
@@
 	(wire
 		(pts
+			(xy 236.22 116.84) (xy 242.57 116.84)
+		)
+		(stroke
+			(width 0)
+			(type default)
+		)
+	)
+	(wire
+		(pts
 			(xy 236.22 88.9) (xy 261.62 88.9)
 		)
@@
 	(wire
 		(pts
+			(xy 242.57 114.3) (xy 236.22 114.3)
+		)
+		(stroke
+			(width 0)
+			(type default)
+		)
+	)
+	(wire
+		(pts
 			(xy 236.22 111.76) (xy 242.57 111.76)
 		)
@@
 	(wire
 		(pts
-			(xy 236.22 121.92) (xy 241.3 121.92)
+			(xy 236.22 121.92) (xy 242.57 121.92)
 		)
 		(stroke
@@
 	(wire
 		(pts
-			(xy 242.57 81.28) (xy 236.22 81.28)
+			(xy 41.91 113.03) (xy 41.91 114.3)
 		)
 		(stroke
@@
 	(wire
 		(pts
-			(xy 41.91 113.03) (xy 41.91 114.3)
+			(xy 256.54 73.66) (xy 256.54 86.36)
 		)
 		(stroke
@@
 	(wire
 		(pts
-			(xy 256.54 73.66) (xy 256.54 86.36)
+			(xy 114.3 185.42) (xy 107.95 185.42)
 		)
 		(stroke
@@
 	(wire
 		(pts
-			(xy 114.3 185.42) (xy 107.95 185.42)
+			(xy 214.63 50.8) (xy 213.36 50.8)
 		)
 		(stroke
@@
 	(wire
 		(pts
-			(xy 214.63 50.8) (xy 213.36 50.8)
+			(xy 49.53 170.18) (xy 54.61 170.18)
 		)
 		(stroke
@@
 	(wire
 		(pts
-			(xy 49.53 170.18) (xy 54.61 170.18)
+			(xy 242.57 119.38) (xy 236.22 119.38)
 		)
 		(stroke
@@
 	(wire
 		(pts
-			(xy 250.19 120.65) (xy 250.19 121.92)
+			(xy 251.46 120.65) (xy 251.46 121.92)
 		)
 		(stroke
@@
 	(wire
 		(pts
-			(xy 242.57 83.82) (xy 236.22 83.82)
-		)
-		(stroke
-			(width 0)
-			(type default)
-		)
-	)
-	(wire
-		(pts
 			(xy 97.79 130.81) (xy 104.14 130.81)
 		)
@@
 	(wire
 		(pts
-			(xy 242.57 78.74) (xy 236.22 78.74)
-		)
-		(stroke
-			(width 0)
-			(type default)
-		)
-	)
-	(wire
-		(pts
 			(xy 97.79 162.56) (xy 96.52 162.56)
 		)
@@
 		)
 	)
+	(label "BUSY"
+		(at 242.57 119.38 180)
+		(effects
+			(font
+				(size 1.27 1.27)
+			)
+			(justify right bottom)
+		)
+	)
 	(label "SCL"
 		(at 247.65 73.66 180)
@@
 		)
 	)
+	(label "DIO1"
+		(at 242.57 114.3 180)
+		(effects
+			(font
+				(size 1.27 1.27)
+			)
+			(justify right bottom)
+		)
+	)
 	(label "CS"
 		(at 82.55 177.8 0)
@@
 		)
 	)
-	(label "DIO1"
-		(at 242.57 83.82 180)
-		(effects
-			(font
-				(size 1.27 1.27)
-			)
-			(justify right bottom)
-		)
-	)
 	(label "MISO"
 		(at 165.1 99.06 0)
@@
 		)
 	)
+	(label "DIO3"
+		(at 242.57 116.84 180)
+		(effects
+			(font
+				(size 1.27 1.27)
+			)
+			(justify right bottom)
+		)
+	)
 	(label "BOOT"
-		(at 236.22 121.92 0)
+		(at 237.49 121.92 0)
 		(effects
 			(font
@@
 		)
 	)
-	(label "BUSY"
-		(at 242.57 78.74 180)
-		(effects
-			(font
-				(size 1.27 1.27)
-			)
-			(justify right bottom)
-		)
-	)
 	(label "ESP_D+"
 		(at 245.11 91.44 180)
@@
 		)
 	)
-	(label "DIO3"
-		(at 242.57 81.28 180)
-		(effects
-			(font
-				(size 1.27 1.27)
-			)
-			(justify right bottom)
-		)
-	)
 	(label "SCK"
 		(at 82.55 185.42 0)
@@
 	(symbol
 		(lib_id "Device:R")
-		(at 245.11 121.92 90)
+		(at 246.38 121.92 90)
 		(mirror x)
 		(unit 1)
@@
 		(dnp no)
 		(property "Reference" "R12"
-			(at 243.84 118.11 90)
+			(at 246.38 117.856 90)
 			(show_name no)
 			(do_not_autoplace no)
@@
 		)
 		(property "Value" "10k"
-			(at 243.84 119.888 90)
+			(at 246.38 119.634 90)
 			(show_name no)
 			(do_not_autoplace no)
@@
 		)
 		(property "Footprint" "Resistor_SMD:R_0402_1005Metric"
-			(at 245.11 120.142 90)
+			(at 246.38 120.142 90)
 			(hide yes)
 			(show_name no)
@@
 		)
 		(property "Datasheet" ""
-			(at 245.11 121.92 0)
+			(at 246.38 121.92 0)
 			(hide yes)
 			(show_name no)
@@
 		)
 		(property "Description" "Resistor"
-			(at 245.11 121.92 0)
+			(at 246.38 121.92 0)
 			(hide yes)
 			(show_name no)
@@
 		)
 		(property "Basic" "Y"
-			(at 245.11 121.92 90)
+			(at 246.38 121.92 90)
 			(hide yes)
 			(show_name no)
@@
 		)
 		(property "JLCPCB Part #" "C25744"
-			(at 245.11 121.92 90)
+			(at 246.38 121.92 90)
 			(hide yes)
 			(show_name no)
@@
 		)
 		(property "Manufacturer" "Uniroyal Elec"
-			(at 245.11 121.92 90)
+			(at 246.38 121.92 90)
 			(hide yes)
 			(show_name no)
@@
 		)
 		(property "Manufacturer Part Number" "0402WGF1002TCE"
-			(at 245.11 121.92 90)
+			(at 246.38 121.92 90)
 			(hide yes)
 			(show_name no)
@@
 	(symbol
 		(lib_id "power:+3V3")
-		(at 250.19 120.65 0)
+		(at 251.46 120.65 0)
 		(unit 1)
 		(body_style 1)
@@
 		(dnp no)
 		(property "Reference" "#PWR063"
-			(at 250.19 124.46 0)
+			(at 251.46 124.46 0)
 			(hide yes)
 			(show_name no)
@@
 		)
 		(property "Value" "+3V3"
-			(at 249.936 116.586 0)
+			(at 251.206 116.586 0)
 			(show_name no)
 			(do_not_autoplace no)
@@
 		)
 		(property "Footprint" ""
-			(at 250.19 120.65 0)
+			(at 251.46 120.65 0)
 			(hide yes)
 			(show_name no)
@@
 		)
 		(property "Datasheet" ""
-			(at 250.19 120.65 0)
+			(at 251.46 120.65 0)
 			(hide yes)
 			(show_name no)
@@
 		)
 		(property "Description" "Power symbol creates a global label with name \"+3V3\""
-			(at 250.19 120.65 0)
+			(at 251.46 120.65 0)
 			(hide yes)
 			(show_name no)

Commit message: pcb: add +3v3 pwr routing
Connections:
- net RGB1: now also U4.33 (GPIO23); no longer U4.34 (GPIO24)
- net RST: now also U4.34 (GPIO24); no longer U4.33 (GPIO23)
Changed lines of the file:
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@@
+		)
+	)
+	(label "RGB1"
+		(at 242.57 109.22 180)
+		(effects
+			(font
+				(size 1.27 1.27)
+			)
+			(justify right bottom)
 		)
 	)
@@
 		)
 	)
-	(label "RST"
-		(at 242.57 109.22 180)
-		(effects
-			(font
-				(size 1.27 1.27)
-			)
-			(justify right bottom)
-		)
-	)
 	(label "MISO"
 		(at 165.1 99.06 0)
@@
 		)
 	)
-	(label "RGB1"
-		(at 242.57 111.76 180)
-		(effects
-			(font
-				(size 1.27 1.27)
-			)
-			(justify right bottom)
-		)
-	)
 	(label "DIO3"
 		(at 114.3 180.34 180)
@@
 		)
 	)
+	(label "RST"
+		(at 242.57 111.76 180)
+		(effects
+			(font
+				(size 1.27 1.27)
+			)
+			(justify right bottom)
+		)
+	)

Commit message: pcb: route boot and rst
Connections:
- net +3V3: now also U4.10 (GPIO1/XTAL_32K_N/ADC1_CH0), U4.9 (GPIO0/XTAL_32K_P)
- no-connect marks 11 -> 9
Changed lines of the file:
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@@
 	)
 	(junction
+		(at 168.91 78.74)
+		(diameter 0)
+		(color 0 0 0 0)
+	)
+	(junction
 		(at 45.72 160.02)
 		(diameter 0)
@@
 	)
 	(no_connect
-		(at 170.18 81.28)
-	)
-	(no_connect
 		(at 114.3 100.33)
 	)
@@
 	)
 	(no_connect
-		(at 170.18 78.74)
-	)
-	(no_connect
 		(at 236.22 99.06)
 	)
@@
 	(wire
 		(pts
+			(xy 168.91 78.74) (xy 168.91 81.28)
+		)
+		(stroke
+			(width 0)
+			(type default)
+		)
+	)
+	(wire
+		(pts
 			(xy 203.2 127) (xy 203.2 128.27)
 		)
@@
 	(wire
 		(pts
+			(xy 168.91 78.74) (xy 170.18 78.74)
+		)
+		(stroke
+			(width 0)
+			(type default)
+		)
+	)
+	(wire
+		(pts
 			(xy 195.58 54.61) (xy 195.58 55.88)
 		)
@@
 	(wire
 		(pts
+			(xy 168.91 77.47) (xy 168.91 78.74)
+		)
+		(stroke
+			(width 0)
+			(type default)
+		)
+	)
+	(wire
+		(pts
 			(xy 57.15 69.85) (xy 57.15 71.12)
 		)
@@
 	(wire
 		(pts
+			(xy 168.91 81.28) (xy 170.18 81.28)
+		)
+		(stroke
+			(width 0)
+			(type default)
+		)
+	)
+	(wire
+		(pts
 			(xy 236.22 73.66) (xy 240.03 73.66)
 		)
@@
 					(unit 1)
 				)
+			)
+		)
+	)
+	(symbol
+		(lib_id "power:+3V3")
+		(at 168.91 77.47 0)
+		(unit 1)
+		(body_style 1)
+		(exclude_from_sim no)
+		(in_bom yes)
+		(on_board yes)
+		(in_pos_files yes)
+		(dnp no)
+		(property "Reference" "#PWR071"
+			(at 168.91 81.28 0)
+			(hide yes)
+			(show_name no)
+			(do_not_autoplace no)
+			(effects
+				(font
+					(size 1.27 1.27)
+				)
+			)
+		)
+		(property "Value" "+3V3"
+			(at 164.338 76.2 0)
+			(show_name no)
+			(do_not_autoplace no)
+			(effects
+				(font
+					(size 1.27 1.27)
+				)
+			)
+		)
+		(property "Footprint" ""
+			(at 168.91 77.47 0)
+			(hide yes)
+			(show_name no)
+			(do_not_autoplace no)
+			(effects
+				(font
+					(size 1.27 1.27)
+				)
+			)
+		)
+		(property "Datasheet" ""
+			(at 168.91 77.47 0)
+			(hide yes)
+			(show_name no)
+			(do_not_autoplace no)
+			(effects
+				(font
+					(size 1.27 1.27)
+				)
+			)
+		)
+		(property "Description" "Power symbol creates a global label with name \"+3V3\""
+			(at 168.91 77.47 0)
+			(hide yes)
+			(show_name no)
+			(do_not_autoplace no)
+			(effects
+				(font
+					(size 1.27 1.27)
+				)
+			)
+		)
+		(pin "1"
+		)
+		(instances
+			(project "carte-meteo-lora-2"
+				(path "/14cd50fe-ec77-4829-bd74-9322c036cdc1"
+					(reference "#PWR071")
+					(unit 1)
+				)
